Commit message: urdf looks okay, need to do more validation.  Will add rviz config once I get lidar and camera up and running.  updated values for teleop based on new data.  The max may not be correct.

File: gemab_description/urdf/gemab.urdf (robot description, URDF)
Before this commit: robot gemab, 3 links, 2 joints
Links:
- added link base_footprint
- link base_link: geometry visual box size=0.47 0.34 0.020
Joints:
- added joint base_joint: type fixed, parent base_footprint, child base_link, origin xyz=0.0 0.0 0.05 rpy=0 0 0
- joint base_to_wheel_left: axis (none) -> 0 0 1; origin xyz=0 0 0 -> xyz=0.235 -0.185 0.045; type fixed -> continuous
- joint base_to_wheel_right: axis (none) -> 0 0 1; origin xyz=0 0 0 -> xyz=0.235 0.185 0.045; type fixed -> continuous

Commit message: Updating launch files, working on getting lidar up and running

File: gemab_description/urdf/gemab.urdf (robot description, URDF)
Before this commit: robot gemab, 4 links, 3 joints
Links:
- added link base_scan; visual cylinder length=0.005 radius=0.04
Joints:
- added joint base_to_laser: type fixed, parent base_link, child base_scan, origin xyz=0.0 0.0 0.1

Commit message: updated urdf with actual measurements

File: gemab_description/urdf/gemab.urdf (robot description, URDF)
Before this commit: robot gemab, 5 links, 4 joints
Joints:
- joint base_joint: origin xyz=0.0 0.0 0.05 rpy=0 0 0 -> xyz=0.0 0.0 0.0 rpy=0 0 0
- joint base_to_laser: origin xyz=0.0 0.0 0.1 -> xyz=35.0 0.0 0.0255
- joint base_to_wheel_left: origin xyz=0.235 -0.185 0.045 -> xyz=0.178 -0.185 -0.0205
- joint base_to_wheel_right: origin xyz=0.235 0.185 0.045 -> xyz=0.178 0.185 -0.0205

Commit message: working on the robot to drive around, need to add the rviz file and add current monitoring

File: gemab_description/urdf/gemab.urdf (robot description, URDF)
Before this commit: robot gemab, 5 links, 4 joints
Links:
- link wheel_left: geometry visual cylinder length=0.01 radius=0.045
- link wheel_right: geometry visual cylinder length=0.01 radius=0.045
Joints:
- joint base_joint: origin xyz=0.0 0.0 0.05 rpy=0 0 0 -> xyz=0.0 0.0 0.0 rpy=0 0 0
- joint base_to_laser: origin xyz=0.0 0.0 0.1 -> xyz=.035 0.0 0.0255
- joint base_to_wheel_left: origin xyz=0.235 -0.185 0.045 -> xyz=0.178 -0.185 -0.0205
- joint base_to_wheel_right: origin xyz=0.235 0.185 0.045 -> xyz=0.178 0.185 -0.0205
